File: cad/eqprop-xor/eqprop-xor.kicad_sch (KiCad schematic)
At the start: 117 parts, among them J1 USB_C_Receptacle_USB2.0_14P, SW1 SW_SPDT, SW2 SW_SPDT, U1 MCP6004, U10 MCP4251-xxxx-P, U11 MCP4251-xxxx-P, U12 MCP4251-xxxx-P, U13 MCP4251-xxxx-P, U14 MCP4822, U15 MCP6002-xP, U16 ADS1115IDGS, U2 LM324, U3 Arduino_Nano_v3.x, U4 CD4053B, U5 CD4053B, U6 MCP4251-xxxx-P, U7 MCP4251-xxxx-P, U8 MCP4251-xxxx-P, U9 MCP4251-xxxx-P

Commit message: Started PCB design
Parts:
- C1, C12, C13: footprint (none) -> Capacitor_THT:CP_Radial_D6.3mm_P2.50mm
- C10, C11, C14, C15, C16, C17, C18, C19, C2, C20, C21, C22, C23, C24, C25, C26, C3, C4, C5, C6, C7, C8, C9: footprint (none) -> Capacitor_SMD:C_0805_2012Metric
- D_GRN1: renamed from D_GRN; value LED -> Green 3mm; footprint (none) -> LED_THT:LED_D3.0mm
- D_GRN2: renamed from D5; value LED -> Green 3mm; footprint (none) -> LED_THT:LED_D3.0mm
- D_PWR1: renamed from D_PWR; footprint (none) -> LED_THT:LED_D3.0mm
- J1: footprint (none) -> Connector_USB:USB_C_Receptacle_GCT_USB4085
- R1, R10, R11, R12, R13, R14, R15, R16, R17, R18, R19, R2, R20, R21, R3, R4, R5, R6, R7, R8, R9, R_CC1, R_CC2, R_H1, R_H2, R_H3, R_H4, R_H5, R_H6, R_H7, R_H8, R_LED1, R_SW1, R_SW2, R_W1, R_W10, R_W11, R_W12, R_W13, R_W14, R_W15, R_W16, R_W2, R_W3, R_W4, R_W5, R_W6, R_W7, R_W8, R_W9: footprint (none) -> Resistor_SMD:R_0805_2012Metric
- R_LED_G1: renamed from R_LED_G; footprint (none) -> Resistor_SMD:R_0805_2012Metric
- R_LED_R1: renamed from R_LED_R; footprint (none) -> Resistor_SMD:R_0805_2012Metric
- R_SET_A1: renamed from R_SET_A; footprint (none) -> Resistor_SMD:R_0805_2012Metric
- R_SET_B1: renamed from R_SET_B; footprint (none) -> Resistor_SMD:R_0805_2012Metric
- SW1, SW2: footprint (none) -> Button_Switch_THT:SW_E-Switch_EG1271_SPDT
- TP1, TP10, TP11, TP2, TP3, TP4, TP5, TP6, TP7, TP8, TP9: footprint (none) -> TestPoint:TestPoint_Pad_1.0x1.0mm
- U1, U2: footprint (none) -> Package_DIP:DIP-14_W7.62mm_Socket
- U10, U11, U12, U13, U6, U7, U8, U9: footprint Package_DIP:DIP-14_W7.62mm -> Package_DIP:DIP-14_W7.62mm_Socket
- U14, U15: footprint (none) -> Package_DIP:DIP-8_W7.62mm_Socket
- U4, U5: footprint (none) -> Package_DIP:DIP-16_W7.62mm_Socket
Connections:
- net +5V: now also C26.1
- net GND: now also C26.2
Other:
- note added: "MEASUREMENT (16-bit ADC)"
- moved on the sheet: C26, R20, R21, U16

Commit message: Complete B.1 EqProp PCB and document fabrication and firmware handoff
Parts:
- removed C1, C12, C13: 100µF, Capacitor_THT:CP_Radial_D6.3mm_P2.50mm, symbol Device:C_Polarized
- removed C10, C11, C14, C15, C16, C17, C18, C19, C2, C20, C21, C22, C23, C24, C25, C26, C3, C5, C7, C9: 100nF, Capacitor_SMD:C_0805_2012Metric, symbol Device:C
- removed C4, C6, C8: 10µF, Capacitor_SMD:C_0805_2012Metric, symbol Device:C_Polarized
- removed D1, D2, D3, D4: BAT42, Diode_THT:D_DO-35_SOD27_P7.62mm_Horizontal, symbol Diode:BAT42
- removed D_GRN1, D_GRN2, D_PWR1: Green 3mm, LED_THT:LED_D3.0mm, symbol Device:LED
- removed J1: USB_C_Receptacle_USB2.0_14P, Connector_USB:USB_C_Receptacle_GCT_USB4085, symbol Connector:USB_C_Receptacle_USB2.0_14P
- removed R1, R10, R11, R12, R13, R14, R15, R2, R7, R8, R9, R_H1, R_H2, R_H3, R_H4, R_H5, R_H6, R_H7, R_H8, R_SW1, R_SW2: 10kΩ, Resistor_SMD:R_0805_2012Metric, symbol Device:R
- removed R16, R17, R18, R19: 0Ω, Resistor_SMD:R_0805_2012Metric, symbol Device:R
- removed R20, R21: 4.7kΩ, Resistor_SMD:R_0805_2012Metric, symbol Device:R
- removed R3, R6: 33kΩ, Resistor_SMD:R_0805_2012Metric, symbol Device:R
- removed R4, R5: 8.2kΩ, Resistor_SMD:R_0805_2012Metric, symbol Device:R
- removed R_CC1, R_CC2: 5.1kΩ, Resistor_SMD:R_0805_2012Metric, symbol Device:R
- removed R_LED1: 1kΩ, Resistor_SMD:R_0805_2012Metric, symbol Device:R
- removed R_LED_G1, R_LED_R1: 470Ω, Resistor_SMD:R_0805_2012Metric, symbol Device:R
- removed R_SET_A1, R_SET_B1: 1MΩ, Resistor_SMD:R_0805_2012Metric, symbol Device:R
- removed R_W1, R_W10, R_W11, R_W12, R_W13, R_W14, R_W15, R_W16, R_W2, R_W3, R_W4, R_W5, R_W6, R_W7, R_W8, R_W9: 1.21kΩ, Resistor_SMD:R_0805_2012Metric, symbol Device:R
- removed SW1, SW2: SW_SPDT, Button_Switch_THT:SW_E-Switch_EG1271_SPDT, symbol Switch:SW_SPDT
- removed TP1, TP10, TP11, TP2, TP3, TP4, TP5, TP6, TP7, TP8, TP9: TestPoint, TestPoint:TestPoint_Pad_1.0x1.0mm, symbol Connector:TestPoint
- removed U1: MCP6004, Package_DIP:DIP-14_W7.62mm_Socket, symbol Amplifier_Operational:MCP6004
- removed U10, U11, U12, U13, U6, U7, U8, U9: MCP4251-xxxx-P, Package_DIP:DIP-14_W7.62mm_Socket, symbol Potentiometer_Digital:MCP4251-xxxx-P
- removed U14: MCP4822, Package_DIP:DIP-8_W7.62mm_Socket, symbol Analog_DAC:MCP4822
- removed U15: MCP6002-xP, Package_DIP:DIP-8_W7.62mm_Socket, symbol Amplifier_Operational:MCP6002-xP
- removed U16: ADS1115IDGS, Package_SO:TSSOP-10_3x3mm_P0.5mm, symbol Analog_ADC:ADS1115IDGS
- removed U2: LM324, Package_DIP:DIP-14_W7.62mm_Socket, symbol Amplifier_Operational:LM324
- removed U3: Arduino_Nano_v3.x, Module:Arduino_Nano, symbol MCU_Module:Arduino_Nano_v3.x
- removed U4, U5: CD4053B, Package_DIP:DIP-16_W7.62mm_Socket, symbol Analog_Switch:CD4053B
Connections:
- no-connect marks 14 -> 0
Other:
- added sheet Balanced nudge current sources (nudge.kicad_sch)
- added sheet Buffered measurement and classifier (measurement.kicad_sch)
- added sheet Buffered voltage references (references.kicad_sch)
- added sheet Complementary input selection (inputs.kicad_sch)
- added sheet Hidden-node activation (activation.kicad_sch)
- added sheet Nano and operator controls (io.kicad_sch)
- added sheet Sixteen programmable weights (weights.kicad_sch)
- added sheet USB power and protection (power.kicad_sch)
- note added: "EqProp XOR — schematic and PCB must be reviewed together. Global labels connect the functional sheets. Manufacturing release requires final ERC, DRC and BOM review."
- note removed: "Bulk decoupling near analog ICs"
- note removed: "Bulk decoupling near digital ICs"
- note removed: "CS pull-ups (deselect SPI during boot)"
- note removed: "INPUT MULTIPLEXERS"
- note removed: "Inference mode toggle switches"
- note removed: "MEASUREMENT (16-bit ADC)"
- note removed: "MICROCONTROLLER"
- note removed: "NUDGE CURRENT INJECTION"
- note removed: "POWER + VOLTAGE REFERENCES"
- note removed: "WEIGHT NETWORK"
- title: (none) -> EqProp XOR — SMD revision
